File: Adapter.sch (KiCad schematic (older format))
At the start: 5 parts

Commit message: More elements.
Parts:
- added J?: CONN_01X03, symbol CONN_01X03
- D?: value LED -> LED_AMBER
- D?: value LED -> LED_GREEN
Connections:
- net 12V: now also D?.2 (A)
- net GND: now also R?.2, J?.3 (P3)
- net PSON: now also D?.2 (A)
- net RTN: now also R?.2
- net SCL: now also J?.1 (P1)
- net SDA: now also J?.2 (P2)
- net at D?.1 (K): now also R?.1 (x2)
Changed lines of the file:
@@
 P 5450 1600
 F 0 "D?" H 5450 1700 50  0000 C CNN
-F 1 "LED" H 5450 1500 50  0000 C CNN
+F 1 "LED_AMBER" H 5450 1500 50  0000 C CNN
 F 2 "" H 5450 1600 50  0001 C CNN
 F 3 "" H 5450 1600 50  0001 C CNN
@@
 P 5450 2000
 F 0 "D?" H 5450 2100 50  0000 C CNN
-F 1 "LED" H 5450 1900 50  0000 C CNN
+F 1 "LED_GREEN" H 5450 1900 50  0000 C CNN
 F 2 "" H 5450 2000 50  0001 C CNN
 F 3 "" H 5450 2000 50  0001 C CNN
@@
 Text GLabel 4600 2000 0    60   Input ~ 0
 RTN
+Text GLabel 5800 2000 2    60   Input ~ 0
+12V
+Text GLabel 5800 1600 2    60   Input ~ 0
+PSON
+Wire Wire Line
+	4600 1600 4800 1600
+Wire Wire Line
+	5100 1600 5300 1600
+Wire Wire Line
+	5600 1600 5800 1600
+Wire Wire Line
+	4600 2000 4800 2000
+Wire Wire Line
+	5100 2000 5300 2000
+Wire Wire Line
+	5600 2000 5800 2000
+$Comp
+L CONN_01X03 J?
+U 1 1 594513DD
+P 5400 2950
+F 0 "J?" H 5400 3150 50  0000 C CNN
+F 1 "CONN_01X03" V 5500 2950 50  0000 C CNN
+F 2 "" H 5400 2950 50  0001 C CNN
+F 3 "" H 5400 2950 50  0001 C CNN
+	1    5400 2950
+	1    0    0    -1
+$EndComp
+Text GLabel 4750 2750 0    60   Input ~ 0
+SCL
+Text GLabel 4750 2950 0    60   Input ~ 0
+SDA
+Text GLabel 4750 3150 0    60   Input ~ 0
+GND
+Wire Wire Line
+	4750 3150 5200 3150
+Wire Wire Line
+	5200 3150 5200 3050
+Wire Wire Line
+	5200 2950 4750 2950
+Wire Wire Line
+	4750 2750 5200 2750
+Wire Wire Line
+	5200 2750 5200 2850
 $EndSCHEMATC

Commit message: WIP
Parts:
- removed J?: CONN_02X32, symbol CONN_02X32
- added J1: PSU_CONNECTOR, symbol PSU_CONNECTOR-RESCUE-Adapter
- added J3, J4, J5, J6, J7, J8: CONN_02X04, symbol CONN_02X04
- added SW1: SW_SPST, symbol SW_SPST
- D1, D2: renamed from D?; footprint (none) -> LEDs:LED-5MM
- gave numbers to parts that had none: 3
Connections:
- net 12V: now also J1.1 (12V), J1.10 (12V), J1.11 (12V), J1.12 (12V), J1.13 (12V), J1.2 (12V), J1.3 (12V), J1.4 (12V), J1.5 (12V), J1.52 (12V), J1.53 (12V), J1.54 (12V), J1.55 (12V), J1.56 (12V), J1.57 (12V), J1.58 (12V), J1.59 (12V), J1.6 (12V), J1.60 (12V), J1.61 (12V), J1.62 (12V), J1.7 (12V), J1.8 (12V), J1.9 (12V), J3.1 (P1), J3.2 (P2), J3.3 (P3), J4.1 (P1), J4.2 (P2), J4.3 (P3), J5.1 (P1), J5.2 (P2), J5.3 (P3), J6.1 (P1), J6.2 (P2), J6.3 (P3), J7.1 (P1), J7.2 (P2), J7.3 (P3), J8.1 (P1), J8.2 (P2), J8.3 (P3)
- net 12VSB: now also D1.2 (A), J1.37 (12VSB)
- net ADDR: now also J1.27 (ADDR)
- net GND: now also J1.30 (GND); no longer R1.2
- net PSINTERRUPT: now also J1.38 (PSINTERRUPT)
- net PSOK: now also J1.35 (PSOK)
- net PSON: now also J1.33 (/PSON), SW1.1 (A); no longer D1.2 (A)
- net RTN: now also R1.2, J1.14 (RTN), J1.15 (RTN), J1.16 (RTN), J1.17 (RTN), J1.18 (RTN), J1.19 (RTN), J1.20 (RTN), J1.21 (RTN), J1.22 (RTN), J1.23 (RTN), J1.24 (RTN), J1.25 (RTN), J1.26 (RTN), J1.39 (RTN), J1.40 (RTN), J1.41 (RTN), J1.42 (RTN), J1.43 (RTN), J1.44 (RTN), J1.45 (RTN), J1.46 (RTN), J1.47 (RTN), J1.48 (RTN), J1.49 (RTN), J1.50 (RTN), J1.51 (RTN), J3.4 (P4), J3.5 (P5), J3.6 (P6), J3.7 (P7), J3.8 (P8), J4.4 (P4), J4.5 (P5), J4.6 (P6), J4.7 (P7), J4.8 (P8), J5.4 (P4), J5.5 (P5), J5.6 (P6), J5.7 (P7), J5.8 (P8), J6.4 (P4), J6.5 (P5), J6.6 (P6), J6.7 (P7), J6.8 (P8), J7.4 (P4), J7.5 (P5), J7.6 (P6), J7.7 (P7), J7.8 (P8), J8.4 (P4), J8.5 (P5), J8.6 (P6), J8.7 (P7), J8.8 (P8), SW1.2 (B)
- net SCL: now also J1.32 (SCL)
- net SDA: now also J1.31 (SDA)

Commit message: Work in progress.
Parts:
- J1: footprint (none) -> psu_connector:COMMON_SLOT_PSU
- J2: footprint (none) -> Pin_Headers:Pin_Header_Angled_1x03_Pitch2.54mm
- J3, J4, J5, J6, J7, J8: footprint (none) -> Connectors_Molex:Molex_MiniFit-JR-5556-08A_2x04x4.20mm_Straight
- R1, R2: footprint (none) -> Resistors_THT:Resistor_Horizontal_RM15mm
- SW1: footprint (none) -> Buttons_Switches_THT:SW_PUSH
Changed lines of the file:
@@
 EESchema Schematic File Version 2
-LIBS:Adapter-rescue
+LIBS:psu_connector
 LIBS:power
 LIBS:device
@@
 LIBS:zetex
 LIBS:Zilog
-LIBS:psu_connector
 LIBS:Adapter-cache
 EELAYER 25 0
@@
 F 0 "R1" V 5030 1600 50  0000 C CNN
 F 1 "560" V 4950 1600 50  0000 C CNN
-F 2 "" V 4880 1600 50  0001 C CNN
+F 2 "Resistors_THT:Resistor_Horizontal_RM15mm" V 4880 1600 50  0001 C CNN
 F 3 "" H 4950 1600 50  0001 C CNN
 	1    4950 1600
@@
 F 0 "R2" V 5030 2000 50  0000 C CNN
 F 1 "560" V 4950 2000 50  0000 C CNN
-F 2 "" V 4880 2000 50  0001 C CNN
+F 2 "Resistors_THT:Resistor_Horizontal_RM15mm" V 4880 2000 50  0001 C CNN
 F 3 "" H 4950 2000 50  0001 C CNN
 	1    4950 2000
@@
 F 0 "J2" H 5400 3150 50  0000 C CNN
 F 1 "CONN_01X03" V 5500 2950 50  0000 C CNN
-F 2 "" H 5400 2950 50  0001 C CNN
+F 2 "Pin_Headers:Pin_Header_Angled_1x03_Pitch2.54mm" H 5400 2950 50  0001 C CNN
 F 3 "" H 5400 2950 50  0001 C CNN
 	1    5400 2950
@@
 F 0 "J3" H 7450 3800 50  0000 C CNN
 F 1 "CONN_02X04" H 7450 3300 50  0000 C CNN
-F 2 "" H 7450 2350 50  0001 C CNN
+F 2 "Connectors_Molex:Molex_MiniFit-JR-5556-08A_2x04x4.20mm_Straight" H 7450 2350 50  0001 C CNN
 F 3 "" H 7450 2350 50  0001 C CNN
 	1    7450 3550
@@
 F 0 "J5" H 8550 3800 50  0000 C CNN
 F 1 "CONN_02X04" H 8550 3300 50  0000 C CNN
-F 2 "" H 8550 2350 50  0001 C CNN
+F 2 "Connectors_Molex:Molex_MiniFit-JR-5556-08A_2x04x4.20mm_Straight" H 8550 2350 50  0001 C CNN
 F 3 "" H 8550 2350 50  0001 C CNN
 	1    8550 3550
@@
 F 0 "J7" H 9650 3800 50  0000 C CNN
 F 1 "CONN_02X04" H 9650 3300 50  0000 C CNN
-F 2 "" H 9650 2350 50  0001 C CNN
+F 2 "Connectors_Molex:Molex_MiniFit-JR-5556-08A_2x04x4.20mm_Straight" H 9650 2350 50  0001 C CNN
 F 3 "" H 9650 2350 50  0001 C CNN
 	1    9650 3550
@@
 F 0 "J4" H 7450 5000 50  0000 C CNN
 F 1 "CONN_02X04" H 7450 4500 50  0000 C CNN
-F 2 "" H 7450 3550 50  0001 C CNN
+F 2 "Connectors_Molex:Molex_MiniFit-JR-5556-08A_2x04x4.20mm_Straight" H 7450 3550 50  0001 C CNN
 F 3 "" H 7450 3550 50  0001 C CNN
 	1    7450 4750
@@
 F 0 "J6" H 8550 5000 50  0000 C CNN
 F 1 "CONN_02X04" H 8550 4500 50  0000 C CNN
-F 2 "" H 8550 3550 50  0001 C CNN
+F 2 "Connectors_Molex:Molex_MiniFit-JR-5556-08A_2x04x4.20mm_Straight" H 8550 3550 50  0001 C CNN
 F 3 "" H 8550 3550 50  0001 C CNN
 	1    8550 4750
@@
 F 0 "J8" H 9650 5000 50  0000 C CNN
 F 1 "CONN_02X04" H 9650 4500 50  0000 C CNN
-F 2 "" H 9650 3550 50  0001 C CNN
+F 2 "Connectors_Molex:Molex_MiniFit-JR-5556-08A_2x04x4.20mm_Straight" H 9650 3550 50  0001 C CNN
 F 3 "" H 9650 3550 50  0001 C CNN
 	1    9650 4750
@@
 F 0 "SW1" H 5300 3925 50  0000 C CNN
 F 1 "SW_SPST" H 5300 3700 50  0000 C CNN
-F 2 "" H 5300 3800 50  0001 C CNN
+F 2 "Buttons_Switches_THT:SW_PUSH" H 5300 3800 50  0001 C CNN
 F 3 "" H 5300 3800 50  0001 C CNN
 	1    5300 3800
@@
 F 0 "J1" H 2600 5275 50  0000 C CNN
 F 1 "PSU_CONNECTOR" H 2600 1925 50  0000 C CNN
-F 2 "" H 2600 3600 50  0001 C CNN
+F 2 "psu_connector:COMMON_SLOT_PSU" H 2600 3600 50  0001 C CNN
 F 3 "" H 2600 3600 50  0001 C CNN
 	1    2600 3600

Commit message: Further layout work.
Parts:
- added J10, J11, J9: 12V, Connectors_Terminal_Blocks:TerminalBlock_Pheonix_MKDS1.5-3pol, symbol CONN_01X03
- added J12, J13, J14: RTN, Connectors_Terminal_Blocks:TerminalBlock_Pheonix_MKDS1.5-3pol, symbol CONN_01X03
- J3, J4, J5, J6, J7, J8: value CONN_02X04 -> PEG
- R1, R2: footprint Resistors_THT:Resistor_Horizontal_RM15mm -> Resistors_THT:Resistor_Horizontal_RM10mm
Connections:
- net 12V: now also J10.1 (P1), J10.2 (P2), J10.3 (P3), J11.1 (P1), J11.2 (P2), J11.3 (P3), J9.1 (P1), J9.2 (P2), J9.3 (P3)
- net RTN: now also J12.1 (P1), J12.2 (P2), J12.3 (P3), J13.1 (P1), J13.2 (P2), J13.3 (P3), J14.1 (P1), J14.2 (P2), J14.3 (P3)
Changed lines of the file:
@@
 F 0 "R1" V 5030 1600 50  0000 C CNN
 F 1 "560" V 4950 1600 50  0000 C CNN
-F 2 "Resistors_THT:Resistor_Horizontal_RM15mm" V 4880 1600 50  0001 C CNN
+F 2 "Resistors_THT:Resistor_Horizontal_RM10mm" V 4880 1600 50  0001 C CNN
 F 3 "" H 4950 1600 50  0001 C CNN
 	1    4950 1600
@@
 F 0 "R2" V 5030 2000 50  0000 C CNN
 F 1 "560" V 4950 2000 50  0000 C CNN
-F 2 "Resistors_THT:Resistor_Horizontal_RM15mm" V 4880 2000 50  0001 C CNN
+F 2 "Resistors_THT:Resistor_Horizontal_RM10mm" V 4880 2000 50  0001 C CNN
 F 3 "" H 4950 2000 50  0001 C CNN
 	1    4950 2000
@@
 P 7450 3550
 F 0 "J3" H 7450 3800 50  0000 C CNN
-F 1 "CONN_02X04" H 7450 3300 50  0000 C CNN
+F 1 "PEG" H 7450 3300 50  0000 C CNN
 F 2 "Connectors_Molex:Molex_MiniFit-JR-5556-08A_2x04x4.20mm_Straight" H 7450 2350 50  0001 C CNN
 F 3 "" H 7450 2350 50  0001 C CNN
@@
 P 8550 3550
 F 0 "J5" H 8550 3800 50  0000 C CNN
-F 1 "CONN_02X04" H 8550 3300 50  0000 C CNN
+F 1 "PEG" H 8550 3300 50  0000 C CNN
 F 2 "Connectors_Molex:Molex_MiniFit-JR-5556-08A_2x04x4.20mm_Straight" H 8550 2350 50  0001 C CNN
 F 3 "" H 8550 2350 50  0001 C CNN
@@
 P 9650 3550
 F 0 "J7" H 9650 3800 50  0000 C CNN
-F 1 "CONN_02X04" H 9650 3300 50  0000 C CNN
+F 1 "PEG" H 9650 3300 50  0000 C CNN
 F 2 "Connectors_Molex:Molex_MiniFit-JR-5556-08A_2x04x4.20mm_Straight" H 9650 2350 50  0001 C CNN
 F 3 "" H 9650 2350 50  0001 C CNN
@@
 P 7450 4750
 F 0 "J4" H 7450 5000 50  0000 C CNN
-F 1 "CONN_02X04" H 7450 4500 50  0000 C CNN
+F 1 "PEG" H 7450 4500 50  0000 C CNN
 F 2 "Connectors_Molex:Molex_MiniFit-JR-5556-08A_2x04x4.20mm_Straight" H 7450 3550 50  0001 C CNN
 F 3 "" H 7450 3550 50  0001 C CNN
@@
 P 8550 4750
 F 0 "J6" H 8550 5000 50  0000 C CNN
-F 1 "CONN_02X04" H 8550 4500 50  0000 C CNN
+F 1 "PEG" H 8550 4500 50  0000 C CNN
 F 2 "Connectors_Molex:Molex_MiniFit-JR-5556-08A_2x04x4.20mm_Straight" H 8550 3550 50  0001 C CNN
 F 3 "" H 8550 3550 50  0001 C CNN
@@
 P 9650 4750
 F 0 "J8" H 9650 5000 50  0000 C CNN
-F 1 "CONN_02X04" H 9650 4500 50  0000 C CNN
+F 1 "PEG" H 9650 4500 50  0000 C CNN
 F 2 "Connectors_Molex:Molex_MiniFit-JR-5556-08A_2x04x4.20mm_Straight" H 9650 3550 50  0001 C CNN
 F 3 "" H 9650 3550 50  0001 C CNN
@@
 Wire Wire Line
 	4300 2700 4300 2800
+$Comp
+L CONN_01X03 J9
+U 1 1 594AC72C
+P 1000 7300
+F 0 "J9" H 1000 7500 50  0000 C CNN
+F 1 "12V" V 1100 7300 50  0000 C CNN
+F 2 "Connectors_Terminal_Blocks:TerminalBlock_Pheonix_MKDS1.5-3pol" H 1000 7300 50  0001 C CNN
+F 3 "" H 1000 7300 50  0001 C CNN
+	1    1000 7300
+	0    1    1    0
+$EndComp
+$Comp
+L CONN_01X03 J10
+U 1 1 594AC79C
+P 1600 7300
+F 0 "J10" H 1600 7500 50  0000 C CNN
+F 1 "12V" V 1700 7300 50  0000 C CNN
+F 2 "Connectors_Terminal_Blocks:TerminalBlock_Pheonix_MKDS1.5-3pol" H 1600 7300 50  0001 C CNN
+F 3 "" H 1600 7300 50  0001 C CNN
+	1    1600 7300
+	0    1    1    0
+$EndComp
+$Comp
+L CONN_01X03 J11
+U 1 1 594AC8E7
+P 2200 7300
+F 0 "J11" H 2200 7500 50  0000 C CNN
+F 1 "12V" V 2300 7300 50  0000 C CNN
+F 2 "Connectors_Terminal_Blocks:TerminalBlock_Pheonix_MKDS1.5-3pol" H 2200 7300 50  0001 C CNN
+F 3 "" H 2200 7300 50  0001 C CNN
+	1    2200 7300
+	0    1    1    0
+$EndComp
+$Comp
+L CONN_01X03 J12
+U 1 1 594AC95B
+P 2800 7300
+F 0 "J12" H 2800 7500 50  0000 C CNN
+F 1 "RTN" V 2900 7300 50  0000 C CNN
+F 2 "Connectors_Terminal_Blocks:TerminalBlock_Pheonix_MKDS1.5-3pol" H 2800 7300 50  0001 C CNN
+F 3 "" H 2800 7300 50  0001 C CNN
+	1    2800 7300
+	0    1    1    0
+$EndComp
+$Comp
+L CONN_01X03 J13
+U 1 1 594AC9E0
+P 3400 7300
+F 0 "J13" H 3400 7500 50  0000 C CNN
+F 1 "RTN" V 3500 7300 50  0000 C CNN
+F 2 "Connectors_Terminal_Blocks:TerminalBlock_Pheonix_MKDS1.5-3pol" H 3400 7300 50  0001 C CNN
+F 3 "" H 3400 7300 50  0001 C CNN
+	1    3400 7300
+	0    1    1    0
+$EndComp
+$Comp
+L CONN_01X03 J14
+U 1 1 594ACA51
+P 4000 7300
+F 0 "J14" H 4000 7500 50  0000 C CNN
+F 1 "RTN" V 4100 7300 50  0000 C CNN
+F 2 "Connectors_Terminal_Blocks:TerminalBlock_Pheonix_MKDS1.5-3pol" H 4000 7300 50  0001 C CNN
+F 3 "" H 4000 7300 50  0001 C CNN
+	1    4000 7300
+	0    1    1    0
+$EndComp
+Text GLabel 700  6800 1    60   Input ~ 0
+12V
+Text GLabel 2500 6800 1    60   Input ~ 0
+RTN
+Wire Wire Line
+	2500 6800 2500 6900
+Wire Wire Line
+	2500 6900 4100 6900
+Wire Wire Line
+	4100 6900 4100 7100
+Wire Wire Line
+	2700 7100 2700 6900
+Connection ~ 2700 6900
+Wire Wire Line
+	2800 7100 2800 6900
+Connection ~ 2800 6900
+Wire Wire Line
+	2900 6900 2900 7100
+Connection ~ 2900 6900
+Wire Wire Line
+	3300 7100 3300 6900
+Connection ~ 3300 6900
+Wire Wire Line
+	3400 7100 3400 6900
+Connection ~ 3400 6900
+Wire Wire Line
+	3500 7100 3500 6900
+Connection ~ 3500 6900
+Wire Wire Line
+	3900 7100 3900 6900
+Connection ~ 3900 6900
+Wire Wire Line
+	4000 7100 4000 6900
+Connection ~ 4000 6900
+Wire Wire Line
+	700  6800 700  6900
+Wire Wire Line
+	700  6900 2300 6900
+Wire Wire Line
+	2300 6900 2300 7100
+Wire Wire Line
+	900  7100 900  6900
+Connection ~ 900  6900
+Wire Wire Line
+	1000 7100 1000 6900
+Connection ~ 1000 6900
+Wire Wire Line
+	1100 7100 1100 6900
+Connection ~ 1100 6900
+Wire Wire Line
+	1500 7100 1500 6900
+Connection ~ 1500 6900
+Wire Wire Line
+	1600 7100 1600 6900
+Connection ~ 1600 6900
+Wire Wire Line
+	1700 7100 1700 6900
+Connection ~ 1700 6900
+Wire Wire Line
+	2100 7100 2100 6900
+Connection ~ 2100 6900
+Wire Wire Line
+	2200 7100 2200 6900
+Connection ~ 2200 6900
 $EndSCHEMATC

Commit message: Further layout work.
Parts:
- removed J1: PSU_CONNECTOR, psu_connector:COMMON_SLOT_PSU, symbol PSU_CONNECTOR-RESCUE-Adapter
- added J1: PSU_CONNECTOR, psu_connector:COMMON_SLOT_PSU, symbol PSU_CONNECTOR
Connections:
- net 12V: now also J1.1 (12V), J1.10 (12V), J1.11 (12V), J1.12 (12V), J1.13 (12V), J1.2 (12V), J1.3 (12V), J1.4 (12V), J1.5 (12V), J1.52 (12V), J1.53 (12V), J1.54 (12V), J1.55 (12V), J1.56 (12V), J1.57 (12V), J1.58 (12V), J1.59 (12V), J1.6 (12V), J1.60 (12V), J1.61 (12V), J1.62 (12V), J1.63 (12V), J1.64 (12V), J1.7 (12V), J1.8 (12V), J1.9 (12V)
- net 12VSB: now also J1.37 (12VSB)
- net ADDR: now also J1.27 (ADDR)
- net GND: now also J1.30 (GND)
- net PSINTERRUPT: now also J1.38 (PSINTERRUPT)
- net PSOK: now also J1.35 (PSOK)
- net PSON: now also J1.33 (/PSON)
- net RTN: now also J1.14 (RTN), J1.15 (RTN), J1.16 (RTN), J1.17 (RTN), J1.18 (RTN), J1.19 (RTN), J1.20 (RTN), J1.21 (RTN), J1.22 (RTN), J1.23 (RTN), J1.24 (RTN), J1.25 (RTN), J1.26 (RTN), J1.39 (RTN), J1.40 (RTN), J1.41 (RTN), J1.42 (RTN), J1.43 (RTN), J1.44 (RTN), J1.45 (RTN), J1.46 (RTN), J1.47 (RTN), J1.48 (RTN), J1.49 (RTN), J1.50 (RTN), J1.51 (RTN)
- net SCL: now also J1.32 (SCL)
- net SDA: now also J1.31 (SDA)
Changed lines of the file:
@@
 Comment4 ""
 $EndDescr
-Text GLabel 3900 4200 2    60   Input ~ 0
+Text GLabel 3450 4100 2    60   Input ~ 0
 12V
 Text GLabel 1300 2200 0    60   Input ~ 0
@@
 Text GLabel 1300 3500 0    60   Input ~ 0
 RTN
-Text GLabel 3900 2900 2    60   Input ~ 0
+Text GLabel 3450 2800 2    60   Input ~ 0
 RTN
-Text GLabel 3700 2600 2    60   Input ~ 0
+Text GLabel 3250 2500 2    60   Input ~ 0
 12VSB
-Text GLabel 4300 2800 3    60   Input ~ 0
+Text GLabel 3850 2700 3    60   Input ~ 0
 PSINTERRUPT
-Text GLabel 3650 2100 2    60   Input ~ 0
+Text GLabel 1550 5200 0    60   Input ~ 0
 SCL
 Text GLabel 1000 5100 0    60   Input ~ 0
 SDA
-Text GLabel 3900 2200 2    60   Input ~ 0
+Text GLabel 3450 2100 2    60   Input ~ 0
 PSON
 Text GLabel 1300 4700 0    60   Input ~ 0
@@
 Text GLabel 1300 5000 0    60   Input ~ 0
 GND
-Text GLabel 3900 2400 2    60   Input ~ 0
+Text GLabel 3450 2300 2    60   Input ~ 0
 PSOK
 $Comp
@@
 	0    1    1    0
 $EndComp
-$Comp
-L PSU_CONNECTOR-RESCUE-Adapter J1
-U 1 1 5949B0F8
-P 2600 3600
-F 0 "J1" H 2600 5275 50  0000 C CNN
-F 1 "PSU_CONNECTOR" H 2600 1925 50  0000 C CNN
-F 2 "psu_connector:COMMON_SLOT_PSU" H 2600 3600 50  0001 C CNN
-F 3 "" H 2600 3600 50  0001 C CNN
-	1    2600 3600
-	1    0    0    -1
-$EndComp
 Wire Wire Line
 	4600 1600 4800 1600
@@
 Connection ~ 1600 3500
 Wire Wire Line
-	3500 2800 3600 2800
-Wire Wire Line
-	3600 2800 3600 4000
-Wire Wire Line
-	3600 4000 3500 4000
-Wire Wire Line
-	3500 4100 3600 4100
-Wire Wire Line
-	3600 4100 3600 5100
-Wire Wire Line
-	3600 5100 3500 5100
-Wire Wire Line
-	3500 2900 3900 2900
-Connection ~ 3600 2900
-Wire Wire Line
-	3500 3000 3600 3000
-Connection ~ 3600 3000
-Wire Wire Line
-	3500 3100 3600 3100
-Connection ~ 3600 3100
-Wire Wire Line
-	3500 3200 3600 3200
-Connection ~ 3600 3200
-Wire Wire Line
-	3500 3300 3600 3300
-Connection ~ 3600 3300
-Wire Wire Line
-	3500 3400 3600 3400
-Connection ~ 3600 3400
-Wire Wire Line
-	3500 3500 3600 3500
-Connection ~ 3600 3500
-Wire Wire Line
-	3500 3600 3600 3600
-Connection ~ 3600 3600
-Wire Wire Line
-	3500 3700 3600 3700
-Connection ~ 3600 3700
-Wire Wire Line
-	3500 3800 3600 3800
-Connection ~ 3600 3800
-Wire Wire Line
-	3500 3900 3600 3900
-Connection ~ 3600 3900
-Wire Wire Line
-	3500 4200 3900 4200
-Connection ~ 3600 4200
-Wire Wire Line
-	3500 4300 3600 4300
-Connection ~ 3600 4300
-Wire Wire Line
-	3500 4400 3600 4400
-Connection ~ 3600 4400
-Wire Wire Line
-	3500 4500 3600 4500
-Connection ~ 3600 4500
-Wire Wire Line
-	3500 4600 3600 4600
-Connection ~ 3600 4600
-Wire Wire Line
-	3500 4700 3600 4700
-Connection ~ 3600 4700
-Wire Wire Line
-	3500 4800 3600 4800
-Connection ~ 3600 4800
-Wire Wire Line
-	3500 4900 3600 4900
-Connection ~ 3600 4900
-Wire Wire Line
-	3500 5000 3600 5000
-Connection ~ 3600 5000
+	3050 2700 3150 2700
+Wire Wire Line
+	3150 2700 3150 3900
+Wire Wire Line
+	3150 3900 3050 3900
+Wire Wire Line
+	3050 4000 3150 4000
+Wire Wire Line
+	3150 4000 3150 5200
+Wire Wire Line
+	3150 5000 3050 5000
+Wire Wire Line
+	3050 2800 3450 2800
+Connection ~ 3150 2800
+Wire Wire Line
+	3050 2900 3150 2900
+Connection ~ 3150 2900
+Wire Wire Line
+	3050 3000 3150 3000
+Connection ~ 3150 3000
+Wire Wire Line
+	3050 3100 3150 3100
+Connection ~ 3150 3100
+Wire Wire Line
+	3050 3200 3150 3200
+Connection ~ 3150 3200
+Wire Wire Line
+	3050 3300 3150 3300
+Connection ~ 3150 3300
+Wire Wire Line
+	3050 3400 3150 3400
+Connection ~ 3150 3400
+Wire Wire Line
+	3050 3500 3150 3500
+Connection ~ 3150 3500
+Wire Wire Line
+	3050 3600 3150 3600
+Connection ~ 3150 3600
+Wire Wire Line
+	3050 3700 3150 3700
+Connection ~ 3150 3700
+Wire Wire Line
+	3050 3800 3150 3800
+Connection ~ 3150 3800
+Wire Wire Line
+	3050 4100 3450 4100
+Connection ~ 3150 4100
+Wire Wire Line
+	3050 4200 3150 4200
+Connection ~ 3150 4200
+Wire Wire Line
+	3050 4300 3150 4300
+Connection ~ 3150 4300
+Wire Wire Line
+	3050 4400 3150 4400
+Connection ~ 3150 4400
+Wire Wire Line
+	3050 4500 3150 4500
+Connection ~ 3150 4500
+Wire Wire Line
+	3050 4600 3150 4600
+Connection ~ 3150 4600
+Wire Wire Line
+	3050 4700 3150 4700
+Connection ~ 3150 4700
+Wire Wire Line
+	3050 4800 3150 4800
+Connection ~ 3150 4800
+Wire Wire Line
+	3050 4900 3150 4900
+Connection ~ 3150 4900
 Wire Wire Line
 	1700 4700 1300 4700
@@
 	1000 5100 1700 5100
 Wire Wire Line
-	3650 2100 3500 2100
-Wire Wire Line
-	3500 2200 3900 2200
-Wire Wire Line
-	3500 2400 3900 2400
-Wire Wire Line
-	3700 2600 3500 2600
-Wire Wire Line
-	3500 2700 4300 2700
-Wire Wire Line
-	4300 2700 4300 2800
+	3050 2100 3450 2100
+Wire Wire Line
+	3050 2300 3450 2300
+Wire Wire Line
+	3250 2500 3050 2500
+Wire Wire Line
+	3050 2600 3850 2600
+Wire Wire Line
+	3850 2600 3850 2700
 $Comp
 L CONN_01X03 J9
@@
 	2200 7100 2200 6900
 Connection ~ 2200 6900
+$Comp
+L PSU_CONNECTOR J1
+U 1 1 594BC644
+P 2600 3600
+F 0 "J1" H 2600 5275 50  0000 C CNN
+F 1 "PSU_CONNECTOR" H 2600 1700 50  0000 C CNN
+F 2 "psu_connector:COMMON_SLOT_PSU" H 2150 3600 50  0001 C CNN
+F 3 "" H 2150 3600 50  0001 C CNN
+	1    2600 3600
+	1    0    0    -1
+$EndComp
+Wire Wire Line
+	3150 5200 3050 5200
+Connection ~ 3150 5000
+Wire Wire Line
+	3050 5100 3150 5100
+Connection ~ 3150 5100
+Wire Wire Line
+	1550 5200 1700 5200
 $EndSCHEMATC
